Commit message: Semi-working version with custom 4WD controller and updated model

File: description/robot_core.xacro (robot description, xacro)
@@ -2,14 +2,17 @@
 <robot xmlns:xacro="http://www.ros.org/wiki/xacro" >
     <xacro:include filename="inertial_macros.xacro"/>
-    <xacro:property name="chassis_length" value="0.335"/>
-    <xacro:property name="chassis_width" value="0.265"/>
-    <xacro:property name="chassis_height" value="0.138"/>
-    <xacro:property name="chassis_mass" value="1.0"/>
-    <xacro:property name="wheel_radius" value="0.033"/>
-    <xacro:property name="wheel_thickness" value="0.026"/>
-    <xacro:property name="wheel_mass" value="0.05"/>
-    <xacro:property name="wheel_offset_x" value="0.226"/>
-    <xacro:property name="wheel_offset_y" value="0.1485"/>
-    <xacro:property name="wheel_offset_z" value="0.01"/>
+    <!-- Updated chassis properties -->
+    <xacro:property name="chassis_length" value="0.9652"/>      <!-- 38 in -->
+    <xacro:property name="chassis_width" value="0.6604"/>       <!-- 26 in -->
+    <xacro:property name="chassis_height" value="0.138"/>       <!-- kept original unless specified -->
+    <xacro:property name="chassis_mass" value="14.608"/>        <!-- full chassis -->
+    <!-- Updated wheel properties -->
+    <xacro:property name="wheel_radius" value="0.1778"/>        <!-- 7 in -->
+    <xacro:property name="wheel_thickness" value="0.1016"/>     <!-- 4 in -->
+    <xacro:property name="wheel_mass" value="1.977"/>           <!-- wheel + hub + gearbox + motor -->
+    <!-- Updated wheel offsets -->
+    <xacro:property name="wheel_offset_x" value="0.4826"/>      <!-- half of chassis_length -->
+    <xacro:property name="wheel_offset_y" value="0.391"/>       <!-- half of chassis_width -->
+    <xacro:property name="wheel_offset_z" value="0.0889"/>      <!-- ~3.5 in off ground -->
     <material name="white">
         <color rgba="1 1 1 1" />
@@ -58,5 +61,5 @@
             </geometry>
         </collision>
-        <xacro:inertial_box mass="0.5" x="${chassis_length}" y="${chassis_width}" z="${chassis_height}">
+        <xacro:inertial_box mass="${chassis_mass}" x="${chassis_length}" y="${chassis_width}" z="${chassis_height}">
             <origin xyz="${chassis_length/2} 0 ${chassis_height/2}" rpy="0 0 0"/>
         </xacro:inertial_box>
@@ -69,5 +72,5 @@
         <parent link="base_link"/>
         <child link="left_front_wheel"/>
-        <origin xyz="0.05 ${wheel_offset_y} 0" rpy="-${pi/2} 0 0" />
+        <origin xyz="${wheel_offset_x - 0.05} ${wheel_offset_y} 0" rpy="-${pi/2} 0 0" />
         <axis xyz="0 0 1"/>
     </joint>
@@ -90,4 +93,12 @@
     <gazebo reference="left_front_wheel">
         <material>Gazebo/Blue</material>
+        <surface>
+            <friction>
+                <ode>
+                    <mu>2.0</mu>
+                    <mu2>2.0</mu2>
+                </ode>
+            </friction>
+        </surface>
     </gazebo>
     <!-- RIGHT FRONT WHEEL LINK  -->
@@ -95,5 +106,5 @@
         <parent link="base_link"/>
         <child link="right_front_wheel"/>
-        <origin xyz="0.05 ${-wheel_offset_y} 0" rpy="${pi/2} 0 0" />
+        <origin xyz="${wheel_offset_x - 0.05} ${-wheel_offset_y} 0" rpy="${pi/2} 0 0" />
         <axis xyz="0 0 -1"/>
     </joint>
@@ -116,4 +127,12 @@
     <gazebo reference="right_front_wheel">
         <material>Gazebo/Blue</material>
+        <surface>
+            <friction>
+                <ode>
+                    <mu>2.0</mu>
+                    <mu2>2.0</mu2>
+                </ode>
+            </friction>
+        </surface>
     </gazebo>
  <!-- LEFT REAR WHEEL LINK -->
@@ -121,5 +140,5 @@
         <parent link="base_link"/>
         <child link="left_wheel"/>
-        <origin xyz="${0.05 -wheel_offset_x} ${wheel_offset_y} 0" rpy="-${pi/2} 0 0" />
+        <origin xyz="${-wheel_offset_x + 0.05} ${wheel_offset_y} 0" rpy="-${pi/2} 0 0" />
         <axis xyz="0 0 1"/>
     </joint>
@@ -133,5 +152,5 @@
         <collision>
             <geometry>
-                <sphere radius="${wheel_radius}"/>
+                <cylinder radius="${wheel_radius}" length="${wheel_thickness}"/>
             </geometry>
         </collision>
@@ -142,4 +161,12 @@
     <gazebo reference="left_wheel">
         <material>Gazebo/Blue</material>
+        <surface>
+            <friction>
+                <ode>
+                    <mu>2.0</mu>
+                    <mu2>2.0</mu2>
+                </ode>
+            </friction>
+        </surface>
     </gazebo>
     <!-- RIGHT REAR WHEEL LINK  -->
@@ -147,5 +174,5 @@
         <parent link="base_link"/>
         <child link="right_wheel"/>
-        <origin xyz="${0.05 -wheel_offset_x} ${-wheel_offset_y} 0" rpy="${pi/2} 0 0" />
+        <origin xyz="${-wheel_offset_x + 0.05} ${-wheel_offset_y} 0" rpy="${pi/2} 0 0" />
         <axis xyz="0 0 -1"/>
     </joint>
@@ -159,5 +186,5 @@
         <collision>
             <geometry>
-                <sphere radius="${wheel_radius}"/>
+                <cylinder radius="${wheel_radius}" length="${wheel_thickness}"/>
             </geometry>
         </collision>
@@ -168,4 +195,12 @@
     <gazebo reference="right_wheel">
         <material>Gazebo/Blue</material>
+        <surface>
+            <friction>
+                <ode>
+                    <mu>2.0</mu>
+                    <mu2>2.0</mu2>
+                </ode>
+            </friction>
+        </surface>
     </gazebo>
 </robot>

Commit message: debugging attempts :(

File: description/robot_core.xacro (robot description, xacro)
@@ -15,4 +15,11 @@
     <xacro:property name="wheel_offset_y" value="0.391"/>       <!-- half of chassis_width -->
     <xacro:property name="wheel_offset_z" value="0.0889"/>      <!-- ~3.5 in off ground -->
+    <!-- Global contact/friction parameters -->
+    <xacro:property name="wheel_mu" value="1.0"/>
+    <xacro:property name="wheel_mu2" value="1.0"/>
+    <xacro:property name="wheel_kp" value="1000000"/>
+    <xacro:property name="wheel_kd" value="500"/>
+    <xacro:property name="wheel_slip1" value="0.01"/>
+    <xacro:property name="wheel_slip2" value="0.01"/>
     <material name="white">
         <color rgba="1 1 1 1" />
@@ -93,11 +100,15 @@
     <gazebo reference="left_front_wheel">
         <material>Gazebo/Blue</material>
-        <surface>
-            <friction>
-                <ode>
-                    <mu>2.0</mu>
-                    <mu2>2.0</mu2>
-                </ode>
-            </friction>
+        <mu>${wheel_mu}</mu>
+        <mu2>${wheel_mu2}</mu2>
+        <surface>
+            <contact>
+                <ode>
+                    <kp>${wheel_kp}</kp>
+                    <kd>${wheel_kd}</kd>
+                    <slip1>${wheel_slip1}</slip1>
+                    <slip2>${wheel_slip2}</slip2>
+                </ode>
+            </contact>
         </surface>
     </gazebo>
@@ -127,11 +138,15 @@
     <gazebo reference="right_front_wheel">
         <material>Gazebo/Blue</material>
-        <surface>
-            <friction>
-                <ode>
-                    <mu>2.0</mu>
-                    <mu2>2.0</mu2>
-                </ode>
-            </friction>
+        <mu>${wheel_mu}</mu>
+        <mu2>${wheel_mu2}</mu2>
+        <surface>
+            <contact>
+                <ode>
+                    <kp>${wheel_kp}</kp>
+                    <kd>${wheel_kd}</kd>
+                    <slip1>${wheel_slip1}</slip1>
+                    <slip2>${wheel_slip2}</slip2>
+                </ode>
+            </contact>
         </surface>
     </gazebo>
@@ -161,11 +176,15 @@
     <gazebo reference="left_wheel">
         <material>Gazebo/Blue</material>
-        <surface>
-            <friction>
-                <ode>
-                    <mu>2.0</mu>
-                    <mu2>2.0</mu2>
-                </ode>
-            </friction>
+        <mu>${wheel_mu}</mu>
+        <mu2>${wheel_mu2}</mu2>
+        <surface>
+            <contact>
+                <ode>
+                    <kp>${wheel_kp}</kp>
+                    <kd>${wheel_kd}</kd>
+                    <slip1>${wheel_slip1}</slip1>
+                    <slip2>${wheel_slip2}</slip2>
+                </ode>
+            </contact>
         </surface>
     </gazebo>
@@ -195,11 +214,15 @@
     <gazebo reference="right_wheel">
         <material>Gazebo/Blue</material>
-        <surface>
-            <friction>
-                <ode>
-                    <mu>2.0</mu>
-                    <mu2>2.0</mu2>
-                </ode>
-            </friction>
+        <mu>${wheel_mu}</mu>
+        <mu2>${wheel_mu2}</mu2>
+        <surface>
+            <contact>
+                <ode>
+                    <kp>${wheel_kp}</kp>
+                    <kd>${wheel_kd}</kd>
+                    <slip1>${wheel_slip1}</slip1>
+                    <slip2>${wheel_slip2}</slip2>
+                </ode>
+            </contact>
         </surface>
     </gazebo>

File: description/ros2_control.xacro (robot description, xacro)
@@ -1,52 +1,4 @@
 <?xml version="1.0"?>
 <robot xmlns:xacro="http://www.ros.org/wiki/xacro">
-    <xacro:unless value="$(arg sim_mode)">
-        <ros2_control name="RealRobot" type="system">
-            <hardware>
-                <plugin>diffdrive_arduino/DiffDriveArduinoHardware</plugin>
-                <param name="left_wheel_name">left_wheel_joint</param>
-                <param name="right_wheel_name">right_wheel_joint</param>
-                <param name="loop_rate">30</param>
-                <param name="device">/dev/ttyUSB0</param>
-                <param name="baud_rate">57600</param>
-                <param name="timeout_ms">1000</param>
-                <param name="enc_counts_per_rev">3436</param>
-            </hardware>
-            <!-- Rear wheels -->
-            <joint name="left_wheel_joint">
-                <command_interface name="velocity">
-                    <param name="min">-10</param>
-                    <param name="max">10</param>
-                </command_interface>
-                <state_interface name="position"/>
-                <state_interface name="velocity"/>
-            </joint>
-            <joint name="right_wheel_joint">
-                <command_interface name="velocity">
-                    <param name="min">-10</param>
-                    <param name="max">10</param>
-                </command_interface>
-                <state_interface name="position"/>
-                <state_interface name="velocity"/>
-            </joint>
-            <!-- Front wheels -->
-            <joint name="left_front_wheel_joint">
-                <command_interface name="velocity">
-                    <param name="min">-10</param>
-                    <param name="max">10</param>
-                </command_interface>
-                <state_interface name="position"/>
-                <state_interface name="velocity"/>
-            </joint>
-            <joint name="right_front_wheel_joint">
-                <command_interface name="velocity">
-                    <param name="min">-10</param>
-                    <param name="max">10</param>
-                </command_interface>
-                <state_interface name="position"/>
-                <state_interface name="velocity"/>
-            </joint>
-        </ros2_control>
-    </xacro:unless>
     <xacro:if value="$(arg sim_mode)">
         <ros2_control name="GazeboSystem" type="system">
