Commit message: Added code for the depth camera to begin publishing data

File: description/depth_camera.xacro (robot description, xacro)
@@ -4,5 +4,5 @@
         <parent link="chassis"/>
         <child link="camera_link"/>
-        <origin xyz="0.305 0 0.08" rpy="0 0 0"/>
+        <origin xyz="-0.005 0 0.099" rpy="0 0 0"/>
     </joint>
     <link name="camera_link">
@@ -38,9 +38,20 @@
                 </clip>
             </camera>
-            <plugin name="camera_controller" filename="libgazebo_ros_camera.so">
+            <plugin name="camera_controller" filename="libgazebo_ros_depth_camera.so">
+                <!--
+                Additional code was added for the camera to begin sending messages to these topics
+                -->
+                <ros>
+                    <imageTopicName>/camera/image_raw</imateTopicName>
+                    <cameraInfoTopicName>camera_info</cameraInfoTopicName>
+                    <depthImageTopicName>/camera/depth/image_raw</depthImageTopicName>
+                    <pointCloudTopicName>camera/depth/points</pointCloudTopicName>
+                </ros>
                 <frame_name>camera_link_optical</frame_name>
                 <min_depth>0.1</min_depth>
                 <max_depth>100.0</max_depth>
             </plugin>
+            <topic>/camera/depth/points</topic>
+            <topic>/camera/depth/image_raw</topic>
         </sensor>
     </gazebo>
