Commit message: Add working RGBD depth camera with complete documentation
Features:
- RGB color image: /camera/image_raw
- Depth image: /camera/depth/image_raw
- Point cloud: /camera/depth/points
- Camera info: /camera/camera_info

Working visualization in both Gazebo and RViz2:
- RGB images display correctly in color
- Depth images work with manual range settings (0.05-8.0m)
- Point clouds display as 3D scatter plots with proper orientation

Switchable camera system:
- RGB camera (red box) vs Depth camera (blue box)
- Easy switching by commenting/uncommenting in robot.urdf.xacro
- Complete setup instructions in README

Technical implementation:
- Uses rgbd_camera sensor type in Gazebo Harmonic
- Proper topic bridging via ros_gz_image_bridge and ros_gz_bridge
- Fixed coordinate frame issues for point cloud orientation
- 640x480 resolution, 10Hz update rate, 62.4° FOV

🤖 Generated with [Claude Code](https://claude.ai/code)

Co-Authored-By: Claude <noreply@anthropic.com>

File: description/depth_camera.xacro (robot description, xacro)
@@ -4,13 +4,22 @@
         <parent link="chassis"/>
         <child link="camera_link"/>
-        <origin xyz="-0.005 0 0.099" rpy="0 0 0"/>
+        <origin xyz="0.9652 0 0.069" rpy="0 0 0"/>
     </joint>
     <link name="camera_link">
         <visual>
             <geometry>
-                <box size="0.010 0.03 0.03"/>
+                <box size="0.02 0.06 0.02"/>
             </geometry>
-            <material name="red"/>
+            <material name="blue"/>
         </visual>
+        <collision>
+            <geometry>
+                <box size="0.02 0.06 0.02"/>
+            </geometry>
+        </collision>
+        <inertial>
+            <mass value="0.01"/>
+            <inertia ixx="0.000001" ixy="0" ixz="0" iyy="0.000001" iyz="0" izz="0.000001"/>
+        </inertial>
     </link>
     <joint name="camera_optical_joint" type="fixed">
@@ -21,6 +30,6 @@
     <link name="camera_link_optical"></link>
     <gazebo reference="camera_link">
-        <material>Gazebo/Red</material>
-        <sensor name="camera" type="depth">
+        <material>Gazebo/Blue</material>
+        <sensor name="camera" type="rgbd_camera">
             <pose> 0 0 0 0 0 0 </pose>
             <visualize>true</visualize>
@@ -29,8 +38,13 @@
                 <horizontal_fov>1.089</horizontal_fov>
                 <image>
-                    <format>B8G8R8</format>
+                    <format>R8G8B8</format>
                     <width>640</width>
                     <height>480</height>
                 </image>
+                <depth_image>
+                    <format>R_FLOAT32</format>
+                    <width>640</width>
+                    <height>480</height>
+                </depth_image>
                 <clip>
                     <near>0.05</near>
@@ -38,20 +52,6 @@
                 </clip>
             </camera>
-            <plugin name="camera_controller" filename="libgazebo_ros_depth_camera.so">
-                <!--
-                Additional code was added for the camera to begin sending messages to these topics
-                -->
-                <ros>
-                    <imageTopicName>/camera/image_raw</imateTopicName>
-                    <cameraInfoTopicName>camera_info</cameraInfoTopicName>
-                    <depthImageTopicName>/camera/depth/image_raw</depthImageTopicName>
-                    <pointCloudTopicName>camera/depth/points</pointCloudTopicName>
-                </ros>
-                <frame_name>camera_link_optical</frame_name>
-                <min_depth>0.1</min_depth>
-                <max_depth>100.0</max_depth>
-            </plugin>
-            <topic>/camera/depth/points</topic>
-            <topic>/camera/depth/image_raw</topic>
+            <topic>camera</topic>
+            <gz_frame_id>camera_link</gz_frame_id>
         </sensor>
     </gazebo>

Commit message: Add USC Lunabotics arena world and fix camera orientation
- Create new USC arena world (6.8m x 5m) with proper zone markings
- Add green L-shaped starting zone boundary
- Add black excavation/obstacle zone separator line
- Add black L-shaped construction zone boundary
- Add 4 boulder obstacles (30-40cm) in obstacle zone with varying heights
- Add red robot spawn area outline (150cm x 75cm) centered at (1,1)
- Add central rectangular column obstacle
- Fix camera optical frame orientation for proper point cloud display
- Remove deprecated launch files (robot.launch.py, simulation.launch.py)
- Update robot spawn position to (1,1,0.2) in unified bringup
- Improve simulation performance by increasing physics step to 5ms

🤖 Generated with [Claude Code](https://claude.ai/code)

Co-Authored-By: Claude <noreply@anthropic.com>

File: description/depth_camera.xacro (robot description, xacro)
@@ -26,5 +26,5 @@
         <parent link="camera_link"/>
         <child link="camera_link_optical"/>
-        <origin xyz="0 0 0" rpy="${-pi/2} 0 ${-pi/2}"/>
+        <origin xyz="0 0 0" rpy="0 0 0"/>
     </joint>
     <link name="camera_link_optical"></link>
