Commit message: IMU Xacro file has been added (minor color fix for Rviz)

File: description/imu.xacro (robot description, xacro)
@@ -11,5 +11,5 @@
                 <box size="0.02 0.02 0.02"/>
             </geometry>
-            <material name="green"/>
+            <material name="blue"/>
         </visual>
         <collision>
