Commit message: Implement unified simulation/hardware system with conditional launch
MAJOR CHANGES - UNTESTED:
- Add conditional logic to robot.urdf.xacro for sim/hardware mode switching
- Create unified_bringup.launch.py supporting both simulation and hardware
- Update robot state publisher to handle new launch arguments
- Comprehensive README.md updates with both sim and hardware instructions
- Add ros_gz dependencies to package.xml for simulation support

FEATURES:
- Single launch file: unified_bringup.launch.py
- Launch arguments: use_hardware, sim_mode, use_ros2_control, world
- Hardware mode uses ODrive ros2_control with CAN interface
- Simulation mode includes depth camera + IMU sensors
- Conditional sensor loading based on mode
- Updated documentation with launch modes and quick reference

⚠️  WARNING: This unified system has NOT been tested yet.
Both simulation and hardware modes need validation before use.

🤖 Generated with [Claude Code](https://claude.ai/code)

Co-Authored-By: Claude <noreply@anthropic.com>

File: description/robot.urdf.xacro (robot description, xacro)
@@ -1,17 +1,64 @@
 <?xml version="1.0"?>
-<robot xmlns:xacro="http://www.ros.org/wiki/xacro"  name="robot">
+<robot xmlns:xacro="http://www.ros.org/wiki/xacro" name="robot">
     <xacro:arg name="use_ros2_control" default="true"/>
-    <xacro:arg name="sim_mode" default="false"/>
+    <xacro:arg name="sim_mode" default="true"/>
+    <xacro:arg name="use_hardware" default="false"/>
     <xacro:include filename="robot_core.xacro" />
-    <xacro:if value="$(arg use_ros2_control)">
-        <xacro:include filename="ros2_control.xacro" />
+    <!-- Control system selection -->
+    <xacro:if value="$(arg use_hardware)">
+        <!-- Hardware mode: Use ODrive ros2_control hardware interface -->
+        <ros2_control name="RealRobot" type="system">
+            <hardware>
+                <plugin>odrive_ros2_control/ODriveHardwareInterface</plugin>
+                <param name="can_interface">can0</param>
+                <param name="enable_watchdog">true</param>
+                <param name="watchdog_timeout">1.0</param>
+                <param name="update_rate">100</param>
+            </hardware>
+            <joint name="left_wheel_joint">
+                <command_interface name="velocity">
+                    <param name="min">-10.0</param>
+                    <param name="max">10.0</param>
+                </command_interface>
+                <state_interface name="position"/>
+                <state_interface name="velocity"/>
+                <state_interface name="effort"/>
+                <param name="odrive_can_ids">[1, 3]</param>
+                <param name="gear_ratio">1.0</param>
+                <param name="wheel_radius">0.165</param>
+                <param name="direction_multiplier">1.0</param>
+            </joint>
+            <joint name="right_wheel_joint">
+                <command_interface name="velocity">
+                    <param name="min">-10.0</param>
+                    <param name="max">10.0</param>
+                </command_interface>
+                <state_interface name="position"/>
+                <state_interface name="velocity"/>
+                <state_interface name="effort"/>
+                <param name="odrive_can_ids">[2, 4]</param>
+                <param name="gear_ratio">1.0</param>
+                <param name="wheel_radius">0.165</param>
+                <param name="direction_multiplier">-1.0</param>
+            </joint>
+        </ros2_control>
     </xacro:if>
-    <xacro:unless value="$(arg use_ros2_control)">
-        <xacro:include filename="gazebo_control.xacro" />
+    <xacro:unless value="$(arg use_hardware)">
+        <!-- Simulation mode: Use existing control systems -->
+        <xacro:if value="$(arg use_ros2_control)">
+            <xacro:include filename="ros2_control.xacro" />
+        </xacro:if>
+        <xacro:unless value="$(arg use_ros2_control)">
+            <xacro:include filename="gazebo_control.xacro" />
+        </xacro:unless>
     </xacro:unless>
+    <!-- Sensors -->
     <xacro:include filename="lidar.xacro" />
-    <!-- <xacro:include filename="camera.xacro" /> -->
-    <xacro:include filename="depth_camera.xacro" />
-    <xacro:include filename="imu.xacro" />
+    <!-- Simulation-only sensors -->
+    <xacro:if value="$(arg sim_mode)">
+        <!-- <xacro:include filename="camera.xacro" /> -->
+        <xacro:include filename="depth_camera.xacro" />
+        <xacro:include filename="imu.xacro" />
+    </xacro:if>
     <xacro:include filename="face.xacro" />
 </robot>
