Commit message: Implement 3-lidar fusion system with coordinate transformation
- Add left and right side lidars positioned at chassis edges
- Reduce all lidar FOV to ±63.8° (from ±68.8°)
- Create coordinate-aware lidar merger (nodes/lidar_merger.py)
- Add Gazebo bridge configuration for scan_left/scan_right topics
- Implement proper coordinate transformation accounting for physical lidar positions
- Front lidar: [0.9652, 0.0] facing forward
- Left lidar: [0.4826, 0.3302] facing left (90°)
- Right lidar: [0.4826, -0.3302] facing right (-90°)
- Output merged scan on /scan_merged topic with 270° coverage
- Fix offset artifacts by transforming each scan point through proper rotation/translation

🤖 Generated with [Claude Code](https://claude.ai/code)

Co-Authored-By: Claude <noreply@anthropic.com>

File: description/lidar.xacro (robot description, xacro)
@@ -4,5 +4,5 @@
         <parent link="chassis"/>
         <child link="laser_frame"/>
-        <origin xyz="0.122 0 0.35" rpy="0 0 0"/>
+        <origin xyz="0.9652 0 0" rpy="0 0 0"/>
     </joint>
     <link name="laser_frame">
@@ -10,11 +10,4 @@
             <geometry>
                 <cylinder radius="0.05" length="0.04"/>
-            </geometry>
-            <material name="black"/>
-        </visual>
-        <visual>
-            <origin xyz="0 0 -0.1"/>
-            <geometry>
-                <cylinder radius="0.01" length="0.23"/>
             </geometry>
             <material name="black"/>
@@ -34,17 +27,23 @@
             <pose> 0 0 0 0 0 0 </pose>
             <visualize>false</visualize>
-            <update_rate>20</update_rate>
+            <update_rate>10</update_rate>
             <lidar>
                 <scan>
                     <horizontal>
-                        <samples>360</samples>
-                        <min_angle>-3.14</min_angle>
-                        <max_angle>3.14</max_angle>
+                        <samples>90</samples>
+                        <min_angle>-1.1127</min_angle>
+                        <max_angle>1.1127</max_angle>
                     </horizontal>
                 </scan>
                 <range>
-                    <min>0.1</min>
-                    <max>12</max>
+                    <min>0.2</min>
+                    <max>8</max>
+                    <resolution>0.01</resolution>
                 </range>
+                <noise>
+                    <type>gaussian</type>
+                    <mean>0.0</mean>
+                    <stddev>0.02</stddev>
+                </noise>
             </lidar>
             <topic>scan</topic>
@@ -52,3 +51,105 @@
         </sensor>
     </gazebo>
+    <!-- LEFT SIDE LIDAR -->
+    <joint name="left_laser_joint" type="fixed">
+        <parent link="chassis"/>
+        <child link="left_laser_frame"/>
+        <origin xyz="0.4826 0.3302 0" rpy="0 0 1.5708"/>
+    </joint>
+    <link name="left_laser_frame">
+        <visual>
+            <geometry>
+                <cylinder radius="0.05" length="0.04"/>
+            </geometry>
+            <material name="black"/>
+        </visual>
+        <collision>
+            <geometry>
+                <cylinder radius="0.05" length="0.04"/>
+            </geometry>
+        </collision>
+        <xacro:inertial_cylinder mass="0.1" length="0.04" radius="0.05">
+            <origin xyz="0 0 0" rpy="0 0 0"/>
+        </xacro:inertial_cylinder>
+    </link>
+    <gazebo reference="left_laser_frame">
+        <material>Gazebo/Black</material>
+        <sensor name="left_laser" type="gpu_lidar">
+            <pose> 0 0 0 0 0 0 </pose>
+            <visualize>false</visualize>
+            <update_rate>10</update_rate>
+            <lidar>
+                <scan>
+                    <horizontal>
+                        <samples>90</samples>
+                        <min_angle>-1.1127</min_angle>
+                        <max_angle>1.1127</max_angle>
+                    </horizontal>
+                </scan>
+                <range>
+                    <min>0.2</min>
+                    <max>8</max>
+                    <resolution>0.01</resolution>
+                </range>
+                <noise>
+                    <type>gaussian</type>
+                    <mean>0.0</mean>
+                    <stddev>0.02</stddev>
+                </noise>
+            </lidar>
+            <topic>scan_left</topic>
+            <gz_frame_id>left_laser_frame</gz_frame_id>
+        </sensor>
+    </gazebo>
+    <!-- RIGHT SIDE LIDAR -->
+    <joint name="right_laser_joint" type="fixed">
+        <parent link="chassis"/>
+        <child link="right_laser_frame"/>
+        <origin xyz="0.4826 -0.3302 0" rpy="0 0 -1.5708"/>
+    </joint>
+    <link name="right_laser_frame">
+        <visual>
+            <geometry>
+                <cylinder radius="0.05" length="0.04"/>
+            </geometry>
+            <material name="black"/>
+        </visual>
+        <collision>
+            <geometry>
+                <cylinder radius="0.05" length="0.04"/>
+            </geometry>
+        </collision>
+        <xacro:inertial_cylinder mass="0.1" length="0.04" radius="0.05">
+            <origin xyz="0 0 0" rpy="0 0 0"/>
+        </xacro:inertial_cylinder>
+    </link>
+    <gazebo reference="right_laser_frame">
+        <material>Gazebo/Black</material>
+        <sensor name="right_laser" type="gpu_lidar">
+            <pose> 0 0 0 0 0 0 </pose>
+            <visualize>false</visualize>
+            <update_rate>10</update_rate>
+            <lidar>
+                <scan>
+                    <horizontal>
+                        <samples>90</samples>
+                        <min_angle>-1.1127</min_angle>
+                        <max_angle>1.1127</max_angle>
+                    </horizontal>
+                </scan>
+                <range>
+                    <min>0.2</min>
+                    <max>8</max>
+                    <resolution>0.01</resolution>
+                </range>
+                <noise>
+                    <type>gaussian</type>
+                    <mean>0.0</mean>
+                    <stddev>0.02</stddev>
+                </noise>
+            </lidar>
+            <topic>scan_right</topic>
+            <gz_frame_id>right_laser_frame</gz_frame_id>
+        </sensor>
+    </gazebo>
 </robot>
